Commit message: Add Gazebo sim bringup with Nav2 SLAM and mecanum ros2_control

File: urdf/mecanum_bot_v3.urdf.xacro (robot description, xacro)
@@ -1,4 +1,4 @@
 <?xml version="1.0"?>
-<robot name="mecanum_bot" xmlns:xacro="http://www.ros.org/wiki/xacro">
+<robot name="mecanum_bot" xmlns:xacro="http://www.ros.org/wiki/xacro" xmlns:gz="http://gazebosim.org/schema">
   <!-- ======================= -->
   <!-- BASE LINK -->
@@ -21,4 +21,12 @@
       <origin xyz="0 0 0" rpy="0 0 0"/>
     </collision>
+    <!-- Inertial needed for Gazebo physics (box 0.55x0.133x0.121, m=2.0kg).
+         Ignored by robot_state_publisher on real hardware. -->
+    <inertial>
+      <origin xyz="0 0 0" rpy="0 0 0"/>
+      <mass value="2.0"/>
+      <inertia ixx="0.0054" ixy="0.0" ixz="0.0"
+               iyy="0.0529" iyz="0.0" izz="0.0534"/>
+    </inertial>
   </link>
   <!-- ======================= -->
@@ -53,4 +61,11 @@
         <origin xyz="0 0 0" rpy="1.5708 0 0"/>
       </collision>
+      <!-- cylinder r=0.048 h=0.05227, m=0.3kg -->
+      <inertial>
+        <origin xyz="0 0 0" rpy="0 0 0"/>
+        <mass value="0.3"/>
+        <inertia ixx="0.000241" ixy="0.0" ixz="0.0"
+                 iyy="0.000241" iyz="0.0" izz="0.000346"/>
+      </inertial>
     </link>
     <joint name="${prefix}_wheel_joint" type="continuous">
@@ -59,4 +74,7 @@
       <origin xyz="${x_offset} ${y_offset} -0.026" rpy="0 0 0"/>
       <axis xyz="0 1 0"/>
+      <!-- effort/velocity limits required so Gazebo can actuate the joint -->
+      <limit effort="10.0" velocity="30.0"/>
+      <dynamics damping="0.1" friction="0.1"/>
     </joint>
   </xacro:macro>
@@ -80,4 +98,16 @@
       </geometry>
     </visual>
+    <collision>
+      <geometry>
+        <cylinder radius="0.035" length="0.022"/>
+      </geometry>
+    </collision>
+    <!-- RPLidar A1 ~0.19kg -->
+    <inertial>
+      <origin xyz="0 0 0" rpy="0 0 0"/>
+      <mass value="0.19"/>
+      <inertia ixx="0.00007" ixy="0.0" ixz="0.0"
+               iyy="0.00007" iyz="0.0" izz="0.00012"/>
+    </inertial>
   </link>
   <!-- lidar centered on box top surface (x,y = box center) -->
@@ -89,3 +119,148 @@
     <origin xyz="0.0 0.0 0.0765" rpy="0 0 0"/>
   </joint>
+  <!-- ======================= -->
+  <!-- GAZEBO SIMULATION -->
+  <!-- Everything below is only used in Gazebo Sim (gz). robot_state_publisher -->
+  <!-- on real hardware ignores <gazebo> and <ros2_control> tags. -->
+  <!-- ======================= -->
+  <!-- Mecanum wheel friction model: diagonal roller directions let the -->
+  <!-- robot strafe (same pattern as gz_ros2_control_demos mecanum demo) -->
+  <gazebo reference="front_left_wheel_link">
+    <collision>
+      <surface>
+        <friction>
+          <ode>
+            <mu>1.0</mu>
+            <mu2>0.0</mu2>
+            <fdir1 gz:expressed_in="base_link">1 -1 0</fdir1>
+          </ode>
+        </friction>
+      </surface>
+    </collision>
+  </gazebo>
+  <gazebo reference="front_right_wheel_link">
+    <collision>
+      <surface>
+        <friction>
+          <ode>
+            <mu>1.0</mu>
+            <mu2>0.0</mu2>
+            <fdir1 gz:expressed_in="base_link">1 1 0</fdir1>
+          </ode>
+        </friction>
+      </surface>
+    </collision>
+  </gazebo>
+  <gazebo reference="rear_left_wheel_link">
+    <collision>
+      <surface>
+        <friction>
+          <ode>
+            <mu>1.0</mu>
+            <mu2>0.0</mu2>
+            <fdir1 gz:expressed_in="base_link">1 1 0</fdir1>
+          </ode>
+        </friction>
+      </surface>
+    </collision>
+  </gazebo>
+  <gazebo reference="rear_right_wheel_link">
+    <collision>
+      <surface>
+        <friction>
+          <ode>
+            <mu>1.0</mu>
+            <mu2>0.0</mu2>
+            <fdir1 gz:expressed_in="base_link">1 -1 0</fdir1>
+          </ode>
+        </friction>
+      </surface>
+    </collision>
+  </gazebo>
+  <!-- Simulated RPLidar A1: GPU lidar (CPU "lidar" type is not supported
+       by Gz Harmonic's SdfEntityCreator), 360 samples, 0.15m - 12m range
+       like the real A1M8, publishes GZ topic /scan which sim.launch.py
+       bridges to ROS /scan -->
+  <gazebo reference="laser_link">
+    <sensor name="lidar" type="gpu_lidar">
+      <always_on>true</always_on>
+      <visualize>false</visualize>
+      <!-- RPLidar A1 spins at ~5.5Hz; keeps software-rendering load down too -->
+      <update_rate>5.5</update_rate>
+      <topic>/scan</topic>
+      <gz_frame_id>laser_link</gz_frame_id>
+      <ray>
+        <scan>
+          <horizontal>
+            <samples>360</samples>
+            <resolution>1.0</resolution>
+            <min_angle>-3.14159</min_angle>
+            <max_angle>3.14159</max_angle>
+          </horizontal>
+        </scan>
+        <range>
+          <min>0.15</min>
+          <max>12.0</max>
+          <resolution>0.01</resolution>
+        </range>
+        <noise>
+          <type>gaussian</type>
+          <mean>0.0</mean>
+          <stddev>0.01</stddev>
+        </noise>
+      </ray>
+    </sensor>
+  </gazebo>
+  <!-- ros2_control hardware interface for Gazebo (velocity-controlled wheels) -->
+  <ros2_control name="GazeboSimSystem" type="system">
+    <hardware>
+      <plugin>gz_ros2_control/GazeboSimSystem</plugin>
+    </hardware>
+    <joint name="front_left_wheel_joint">
+      <command_interface name="velocity">
+        <param name="min">-30</param>
+        <param name="max">30</param>
+      </command_interface>
+      <state_interface name="position"/>
+      <state_interface name="velocity"/>
+    </joint>
+    <joint name="front_right_wheel_joint">
+      <command_interface name="velocity">
+        <param name="min">-30</param>
+        <param name="max">30</param>
+      </command_interface>
+      <state_interface name="position"/>
+      <state_interface name="velocity"/>
+    </joint>
+    <joint name="rear_left_wheel_joint">
+      <command_interface name="velocity">
+        <param name="min">-30</param>
+        <param name="max">30</param>
+      </command_interface>
+      <state_interface name="position"/>
+      <state_interface name="velocity"/>
+    </joint>
+    <joint name="rear_right_wheel_joint">
+      <command_interface name="velocity">
+        <param name="min">-30</param>
+        <param name="max">30</param>
+      </command_interface>
+      <state_interface name="position"/>
+      <state_interface name="velocity"/>
+    </joint>
+  </ros2_control>
+  <gazebo>
+    <plugin filename="gz_ros2_control-system" name="gz_ros2_control::GazeboSimROS2ControlPlugin">
+      <parameters>$(find my_robot_nav)/config/controllers.yaml</parameters>
+      <ros>
+        <!-- Nav2 speaks Twist on /cmd_vel; twist_stamper (sim.launch.py)
+             republishes it stamped on /cmd_vel_stamped for the controller's
+             ~/reference TwistStamped input; ~/odometry + ~/tf_odometry go
+             straight to /odom + /tf -->
+        <remapping>/mecanum_drive_controller/reference:=/cmd_vel_stamped</remapping>
+        <remapping>/mecanum_drive_controller/odometry:=/odom</remapping>
+        <remapping>/mecanum_drive_controller/tf_odometry:=/tf</remapping>
+      </ros>
+    </plugin>
+  </gazebo>
 </robot>
